File: Hardware/UNO_Q_Breakout/UNO_Q_Breakout.kicad_sch (KiCad schematic)
At the start: 3 parts, among them J1 Conn_02x30_Odd_Even, J2 LAMP1

Commit message: Update boms
Parts:
- J1: Manf# FTSH-130-04-L-DV -> 20021121-00034T4LF
- J2: Manf# (none) -> 84952-6
Changed lines of the file:
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@@
 			)
 		)
-		(property "Manf#" "FTSH-130-04-L-DV"
+		(property "Manf#" "20021121-00034T4LF"
 			(at 144.145 92.71 0)
 			(effects
@@
 			)
 		)
+		(property "Manf#" "84952-6"
+			(at 215.9 74.93 0)
+			(effects
+				(font
+					(size 1.27 1.27)
+				)
+			)
+		)
